Commit message: Added kirby part in urdf

File: src/my_robot_description/urdf/rubot/rubot1_mecanum.urdf (robot description, URDF)
Before this commit: robot rubot, 9 links, 8 joints
Links:
- added link kirby, mass 0.8; collision box size=0.32 0.32 0.32; visual mesh filename=file://$(find my_robot_description)/meshes/rubot/kirby.stl scale=0.04 0.04 0.04
Joints:
- added joint joint_kirby: type fixed, parent base_link, child kirby, origin xyz=0 0 0.155 rpy=0 0 1.57

Commit message: Smaller kirby colision in urdf

File: src/my_robot_description/urdf/rubot/rubot1_mecanum.urdf (robot description, URDF)
Before this commit: robot rubot, 10 links, 9 joints
Links:
- link kirby: geometry collision box size=0.03 0.03 0.03; visual mesh filename=file://$(find my_robot_description)/meshes/rubot/kirby.stl scale=0.04 0.04 0.04
